Commit message: upload

File: urdf/objects/block2.urdf (robot description, URDF)
Before this commit: robot block, 1 links, 0 joints
Links:
- link block: mass 0.00001 -> 0.001

File: urdf/objects/table.urdf (robot description, URDF)
Before this commit: robot table, 1 links, 0 joints
Links:
- link table: geometry collision box size=1 1 0.05; visual box size=1 0.8 0.05
